File: AVPCB.kicad_sch (KiCad schematic)
At the start: 23 parts, among them J1 Screw_Terminal_01x02, J2 Screw_Terminal_01x02, J3 XT90PW-F, J4 Conn_01x04, J5 Conn_01x04, J6 Conn_01x04, J7 Conn_01x02, J8 Conn_01x02, U1 Teensy4.1, U2 SN65HVD230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

Commit message: Add files via upload
Parts:
- removed J1, J2: Screw_Terminal_01x02, symbol Connector:Screw_Terminal_01x02
- added J1, J2: B2B-XH-A, B2B-XH-A*, symbol Connector_Generic:Conn_01x02
- added J10: B2B-XH-A, SamacSys_Parts:B2BXHA, symbol Connector_Generic:Conn_01x02
- added J11: B4B-XH-A, SamacSys_Parts:B4BXHA, symbol Connector_Generic:Conn_01x04
- added J9: B2B-XH-A*, B2B-XH-A*, symbol Connector_Generic:Conn_01x02
- F1, F2, F3: footprint (none) -> SamacSys_Parts:3557-2
- J4, J5, J6: value Conn_01x04 -> B4B-XH-A; footprint (none) -> SamacSys_Parts:B4BXHA
- J7: value Conn_01x02 -> B2B-XH-A; footprint (none) -> SamacSys_Parts:B2BXHA
- J8: value Conn_01x02 -> B2B-XH-A; footprint (none) -> B2B-XH-A*
- PS1: footprint THL_30-4812WI:CONV_THL_30-4812WI -> SamacSys_Parts:THL304812WI
- PS2: footprint THN_20-2411WI:CONV_THN_20-2411WI -> SamacSys_Parts:THN_20WI_SERIES
Connections:
- net 12V: now also PS2.1 (+VIN(VCC))
- net 3.3V: no longer U1.46 (3V3), U4.46 (3V3)
- net 48V: no longer PS2.1 (+VIN(VCC))
- net CANH: now also J1.1 (Pin_1), J2.1 (Pin_1)
- net CANL: now also J1.2 (Pin_2), J2.2 (Pin_2)
- net Enc3.3: now also U1.36 (14_A0_TX3_SPDIF_OUT)
- net GND: now also J10.1 (Pin_1), J10.2 (Pin_2), J11.3 (Pin_3), J11.4 (Pin_4)
- net LSwitch: now also U1.39 (17_A3_TX4_SDA1); no longer U1.2 (0_RX1_CRX2_CS1)
- net RSwitch: now also U1.40 (18_A4_SDA); no longer U1.3 (1_TX1_CTX2_MISO1)
- net PUL+: now reaches U1.37 (15_A1_RX3_SPDIF_IN)
- net DIR+: now reaches U1.38 (16_A2_RX4_SCL1)
- net BrakeEnc: now reaches U4.36 (14_A0_TX3_SPDIF_OUT)
- net BrakeEnc: now also J11.2 (Pin_2)
- net BRAKE_DIR: now reaches U4.40 (18_A4_SDA)
- net BRAKE_PWM: now reaches U4.41 (19_A5_SCL)
- net /BRAKE_DIR: now reaches U4.42 (20_A6_TX5_LRCLK1)
- new net 3.3V_1: U1.46 (3V3)
- new net 3.3V_2: J11.1 (Pin_1), U4.46 (3V3)
- new net BTN8982 Motor Driver/M+: J9.1 (Pin_1)
- new net BTN8982 Motor Driver/M-: J9.2 (Pin_2)
Other:
- added sheet BTN8982 Motor Driver (btn8982.kicad_sch)
- note added: "For stepper driver"
- note added: "Fuse Holder: https://www.digikey.com/en/products/detail/keystone-electronics/3557-2/2137305"
- note added: "Heatsink: https://www.tracopower.com/accessory/thl-hs1"
- note added: "brake"
- note added: "stepper"
- moved on the sheet: U1, U4

Commit message: Add files via upload
Parts:
- removed J3: XT90PW-F, XT90PW-F:AMASS_XT90PW-F, symbol XT90PW-F:XT90PW-F
- removed U1, U4: Teensy4.1, symbol teensy:Teensy4.1
- added IC1, IC2: TEENSY_4.1, TEENSY41, symbol SamacSys_Parts:TEENSY_4.1
- added J3: XT90PW-F, XT90PWF, symbol SamacSys_Parts:XT90PW-F
- D1: footprint (none) -> Diode_SMD:D_0805_2012Metric_Pad1.15x1.40mm_HandSolder
- J1, J2, J8: footprint B2B-XH-A* -> SamacSys_Parts:B2BXHA
- J9: value B2B-XH-A* -> B2B-XH-A; footprint B2B-XH-A* -> SamacSys_Parts:B2BXHA
- R1, R2, R3, R4: footprint (none) -> Resistor_SMD:R_0805_2012Metric_Pad1.20x1.40mm_HandSolder
Connections:
- net 3.3V_1: now also IC1.42 (3.3V_1)
- net 3.3V_2: now also IC2.42 (3.3V_1)
- net 5V: now also IC1.52 (+5V), IC2.52 (+5V)
- net BRAKE_DIR: now also IC2.18 (A4)
- net BRAKE_PWM: now also IC2.19 (A5)
- net BrakeEnc: now also IC2.14 (A0)
- net CRX1_1: now also IC1.23 (A9)
- net CRX1_2: now also IC2.23 (A9)
- net CTX1_1: now also IC1.22 (A8)
- net CTX1_2: now also IC2.22 (A8)
- net DIR+: now also IC1.16 (A2)
- net Enc3.3: now also IC1.14 (A0)
- net GND: now also IC1.45 (GND_1), IC2.45 (GND_1), J3.2 (-)
- net LSwitch: now also IC1.17 (A3)
- net PUL+: now also IC1.15 (A1)
- net RSwitch: now also IC1.18 (A4)
- net /BRAKE_DIR: now also IC2.20 (A6)
- net at F1.1: now also J3.1 (+)
